File: Top_level_schematice.kicad_sch (KiCad schematic)
At the start: 10 parts, among them U1 ESP32-WROOM-32, U2 TMP100, U3 TMP100, U4 TMP100, U5 TMP100, U6 TMP100, U7 TMP100, U8 TMP100, U9 TMP100

Commit message: Add files via upload
Parts:
- added BZ10, BZ2, BZ3, BZ4, BZ5, BZ6, BZ7, BZ8, BZ9: Buzzer, Buzzer_Beeper:Buzzer_12x9.5RM7.6, symbol Device:Buzzer
Connections:
- net GND: now also BZ1.2 (+), BZ10.2 (+), BZ2.2 (+), BZ3.2 (+), BZ4.2 (+), BZ5.2 (+), BZ6.2 (+), BZ7.2 (+), BZ8.2 (+), BZ9.2 (+)
- net at BZ1.1 (-): now also U1.10 (IO25), BZ10.1 (-), BZ2.1 (-), BZ3.1 (-), BZ4.1 (-), BZ5.1 (-), BZ6.1 (-), BZ7.1 (-), BZ8.1 (-), BZ9.1 (-)
